File: schemat_i_inne/7DLIB_AVR/7DLIB_AVR.sch (KiCad schematic (older format))
At the start: 4 parts, among them J1 USBASP, U1 ATtiny2313-20SU, Y1 Crystal 12Mhz

Commit message: Naprawione kolory
Naprawione kolory i schemat pdf dla AVR
Parts:
- removed U1: ATtiny2313-20SU, Package_SO:SOIC-20W_7.5x12.8mm_P1.27mm, symbol MCU_Microchip_ATtiny:ATtiny2313-20SU
- added U?: Attiny2313_fix, symbol AT:Attiny2313_fix
Connections:
- net GND: now also U?.10 (GND)
- net VCC: now also U?.20 (VCC)
- net at J1.6 (Pin_6): now also U?.1 (PA2/~RESET)
- net at U?.5 (G): now also U?.11 (PD6)
- net at U?.14 (DIG1): now also U?.12 (PB0)
- net at U?.11 (DIG2): now also U?.13 (PB1)
- net at U?.10 (DIG3): now also U?.14 (PB2)
- net at U?.6 (DIG4): now also U?.15 (PB3)
- net at J1.3 (Pin_3): now also U?.17 (PB5)
- net at J1.4 (Pin_4): now also U?.18 (PB6)
- net at J1.5 (Pin_5): now also U?.19 (PB7)
- net at U?.13 (A): now also U?.2 (PD0)
- net at U?.9 (B): now also U?.3 (PD1)
- net at Y1.2: now also U?.4 (PA1/XTAL2)
- net at Y1.1: now also U?.5 (PA0/XTAL1)
- net at U?.4 (C): now also U?.6 (PD2)
- net at U?.2 (D): now also U?.7 (PD3)
- net at U?.1 (E): now also U?.8 (PD4)
- net at U?.12 (F): now also U?.9 (PD5)
Changed lines of the file:
@@
 $EndDescr
-$Comp
-L MCU_Microchip_ATtiny:ATtiny2313-20SU U1
-U 1 1 620EA465
-P 3800 4250
-F 0 "U1" H 3800 5531 50  0000 C CNN
-F 1 "ATtiny2313-20SU" H 3800 5440 50  0000 C CNN
-F 2 "Package_SO:SOIC-20W_7.5x12.8mm_P1.27mm" H 3800 4250 50  0001 C CIN
-F 3 "http://ww1.microchip.com/downloads/en/DeviceDoc/Atmel-2543-AVR-ATtiny2313_Datasheet.pdf" H 3800 4250 50  0001 C CNN
-	1    3800 4250
-	1    0    0    -1
-$EndComp
 $Comp
 L power:VCC #PWR02
@@
 	1    0    0    -1
 $EndComp
+$Comp
+L AT:Attiny2313_fix U?
+U 1 1 62589A88
+P 3800 4250
+F 0 "U?" H 3800 5531 50  0000 C CNN
+F 1 "Attiny2313_fix" H 3800 5440 50  0000 C CNN
+F 2 "" H 4050 3750 50  0001 C CNN
+F 3 "" H 4050 3750 50  0001 C CNN
+	1    3800 4250
+	1    0    0    -1
+$EndComp

Commit message: Mniejsze poprawki
mało istotne poprawki kosmetyczne
Parts:
- gave numbers to parts that had none: 2
Changed lines of the file:
@@
 	6200 1900 6200 4150
 $Comp
-L 7SEG:F5463BH-Display_Character U?
+L 7SEG:F5463BH-Display_Character U2
 U 1 1 625499E3
 P 5800 4700
-F 0 "U?" H 5775 5275 50  0000 C CIN
+F 0 "U2" H 5775 5275 50  0000 C CIN
 F 1 "F5463BH-Display_Character" H 5775 5184 50  0000 C CNN
 F 2 "Display_7Segment:F5463BH" H 5850 5250 50  0001 C CNN
@@
 $EndComp
 $Comp
-L AT:Attiny2313_fix U?
+L AT:Attiny2313_fix U1
 U 1 1 62589A88
 P 3800 4250
-F 0 "U?" H 3800 5531 50  0000 C CNN
+F 0 "U1" H 3800 5531 50  0000 C CNN
 F 1 "Attiny2313_fix" H 3800 5440 50  0000 C CNN
 F 2 "" H 4050 3750 50  0001 C CNN
